File: Driver.kicad_pcb (KiCad board)
At the start: 2 copper layers, 58.6 x 36 mm, 54 parts, among them IC1 ESP32-PICO-V3, IC2 LMR36506, IC3 MA702GQ-P, IC4 SN65HVD230QDRG4, J1 XT30PB, U1 DRV8316R

Commit message: Updates
Parts:
- J1: footprint DriverParts:XT30_Combined -> DriverParts:XT30PB
- moved J1 6.37 mm to (119.3, 92.2), turned to 180 degrees
Other:
- board size 58.6 x 36 mm -> 50 x 36 mm
