File: Driver.sch (KiCad schematic (older format))
At the start: 54 parts, among them IC1 ESP32-PICO-V3, IC2 LMR36506, IC3 MA702GQ-P, IC4 SN65HVD230QDRG4, J1 XT30PB, U1 DRV8316R

Commit message: Updates
Parts:
- J1: footprint DriverParts:XT30_Combined -> DriverParts:XT30PB
Changed lines of the file:
@@
 F 0 "J1" H 3928 5496 50  0000 L CNN
 F 1 "XT30PB" H 3928 5405 50  0000 L CNN
-F 2 "DriverParts:XT30_Combined" H 3950 5600 50  0001 L CNN
+F 2 "DriverParts:XT30PB" H 3950 5600 50  0001 L CNN
 F 3 "https://www.tme.eu/Document/4acc913878197f8c2e30d4b8cdc47230/XT30UPB%20SPEC.pdf" H 3950 5500 50  0001 L CNN
 F 4 "Mini XT30 Connector" H 3950 5400 50  0001 L CNN "Description"
